File: pcb/MainBoard/usbc.kicad_sch (KiCad schematic)
At the start: 9 parts

Commit message: pcb progress
Parts:
- D301, D302, D303, D304, D305: renamed from D?; footprint can:DFN1006_TVS -> led-matrix:DFN1006_TVS
- J301: renamed from J?; footprint Connector_USB:USB_C_Receptacle_HRO_TYPE-C-31-M-12 -> led-matrix:USB_C_Receptacle_HRO_TYPE-C-31-M-12
- gave numbers to parts that had none: 3
Changed lines of the file:
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@@
 		(dnp no)
 		(fields_autoplaced yes)
-		(property "Reference" "R?"
+		(property "Reference" "R303"
 			(at 22.86 74.9299 0)
 			(effects
@@
 			(project "MainBoard"
 				(path "/ac576ee3-ac6f-4244-babf-9af36c7a7db3/5232c3be-bd03-4015-929e-0effd1f09850"
-					(reference "R?")
+					(reference "R303")
 					(unit 1)
 				)
@@
 		(dnp no)
 		(fields_autoplaced yes)
-		(property "Reference" "#PWR07"
+		(property "Reference" "#PWR0301"
 			(at 74.93 58.42 0)
 			(effects
@@
 			(project "MainBoard"
 				(path "/ac576ee3-ac6f-4244-babf-9af36c7a7db3/5232c3be-bd03-4015-929e-0effd1f09850"
-					(reference "#PWR07")
+					(reference "#PWR0301")
 					(unit 1)
 				)
@@
 		(dnp no)
 		(fields_autoplaced yes)
-		(property "Reference" "D?"
+		(property "Reference" "D304"
 			(at 123.19 41.275 0)
 			(effects
@@
 			)
 		)
-		(property "Footprint" "can:DFN1006_TVS"
+		(property "Footprint" "led-matrix:DFN1006_TVS"
 			(at 123.19 44.45 0)
 			(effects
@@
 			(project "MainBoard"
 				(path "/ac576ee3-ac6f-4244-babf-9af36c7a7db3/5232c3be-bd03-4015-929e-0effd1f09850"
-					(reference "D?")
+					(reference "D304")
 					(unit 1)
 				)
@@
 		(on_board yes)
 		(dnp no)
-		(property "Reference" "J?"
+		(property "Reference" "J301"
 			(at 30.4165 22.86 0)
 			(effects
@@
 			)
 		)
-		(property "Footprint" "Connector_USB:USB_C_Receptacle_HRO_TYPE-C-31-M-12"
+		(property "Footprint" "led-matrix:USB_C_Receptacle_HRO_TYPE-C-31-M-12"
 			(at 31.75 45.72 0)
 			(effects
@@
 			(project "MainBoard"
 				(path "/ac576ee3-ac6f-4244-babf-9af36c7a7db3/5232c3be-bd03-4015-929e-0effd1f09850"
-					(reference "J?")
+					(reference "J301")
 					(unit 1)
 				)
@@
 		(on_board yes)
 		(dnp no)
-		(property "Reference" "#FLG02"
+		(property "Reference" "#FLG0302"
 			(at 31.115 68.58 0)
 			(effects
@@
 			(project "MainBoard"
 				(path "/ac576ee3-ac6f-4244-babf-9af36c7a7db3/5232c3be-bd03-4015-929e-0effd1f09850"
-					(reference "#FLG02")
+					(reference "#FLG0302")
 					(unit 1)
 				)
@@
 		(dnp no)
 		(fields_autoplaced yes)
-		(property "Reference" "#FLG01"
+		(property "Reference" "#FLG0301"
 			(at 49.53 24.765 0)
 			(effects
@@
 			(project "MainBoard"
 				(path "/ac576ee3-ac6f-4244-babf-9af36c7a7db3/5232c3be-bd03-4015-929e-0effd1f09850"
-					(reference "#FLG01")
+					(reference "#FLG0301")
 					(unit 1)
 				)
@@
 		(dnp no)
 		(fields_autoplaced yes)
-		(property "Reference" "#PWR013"
+		(property "Reference" "#PWR0302"
 			(at 129.54 62.23 0)
 			(effects
@@
 			(project "MainBoard"
 				(path "/ac576ee3-ac6f-4244-babf-9af36c7a7db3/5232c3be-bd03-4015-929e-0effd1f09850"
-					(reference "#PWR013")
+					(reference "#PWR0302")
 					(unit 1)
 				)
@@
 		(dnp no)
 		(fields_autoplaced yes)
-		(property "Reference" "R?"
+		(property "Reference" "R301"
 			(at 71.12 43.1799 0)
 			(effects
@@
 			(project "MainBoard"
 				(path "/ac576ee3-ac6f-4244-babf-9af36c7a7db3/5232c3be-bd03-4015-929e-0effd1f09850"
-					(reference "R?")
+					(reference "R301")
 					(unit 1)
 				)
@@
 		(dnp no)
 		(fields_autoplaced yes)
-		(property "Reference" "D?"
+		(property "Reference" "D301"
 			(at 123.19 22.225 0)
 			(effects
@@
 			)
 		)
-		(property "Footprint" "can:DFN1006_TVS"
+		(property "Footprint" "led-matrix:DFN1006_TVS"
 			(at 123.19 25.4 0)
 			(effects
@@
 			(project "MainBoard"
 				(path "/ac576ee3-ac6f-4244-babf-9af36c7a7db3/5232c3be-bd03-4015-929e-0effd1f09850"
-					(reference "D?")
+					(reference "D301")
 					(unit 1)
 				)
@@
 		(dnp no)
 		(fields_autoplaced yes)
-		(property "Reference" "R?"
+		(property "Reference" "R302"
 			(at 78.74 43.1799 0)
 			(effects
@@
 			(project "MainBoard"
 				(path "/ac576ee3-ac6f-4244-babf-9af36c7a7db3/5232c3be-bd03-4015-929e-0effd1f09850"
-					(reference "R?")
+					(reference "R302")
 					(unit 1)
 				)
@@
 		(dnp no)
 		(fields_autoplaced yes)
-		(property "Reference" "D?"
+		(property "Reference" "D303"
 			(at 123.19 34.925 0)
 			(effects
@@
 			)
 		)
-		(property "Footprint" "can:DFN1006_TVS"
+		(property "Footprint" "led-matrix:DFN1006_TVS"
 			(at 123.19 38.1 0)
 			(effects
@@
 			(project "MainBoard"
 				(path "/ac576ee3-ac6f-4244-babf-9af36c7a7db3/5232c3be-bd03-4015-929e-0effd1f09850"
-					(reference "D?")
+					(reference "D303")
 					(unit 1)
 				)
@@
 		(dnp no)
 		(fields_autoplaced yes)
-		(property "Reference" "#PWR010"
+		(property "Reference" "#PWR0304"
 			(at 20.32 88.9 0)
 			(effects
@@
 			(project "MainBoard"
 				(path "/ac576ee3-ac6f-4244-babf-9af36c7a7db3/5232c3be-bd03-4015-929e-0effd1f09850"
-					(reference "#PWR010")
+					(reference "#PWR0304")
 					(unit 1)
 				)
@@
 		(dnp no)
 		(fields_autoplaced yes)
-		(property "Reference" "D?"
+		(property "Reference" "D302"
 			(at 123.19 28.575 0)
 			(effects
@@
 			)
 		)
-		(property "Footprint" "can:DFN1006_TVS"
+		(property "Footprint" "led-matrix:DFN1006_TVS"
 			(at 123.19 31.75 0)
 			(effects
@@
 			(project "MainBoard"
 				(path "/ac576ee3-ac6f-4244-babf-9af36c7a7db3/5232c3be-bd03-4015-929e-0effd1f09850"
-					(reference "D?")
+					(reference "D302")
 					(unit 1)
 				)
@@
 		(dnp no)
 		(fields_autoplaced yes)
-		(property "Reference" "D?"
+		(property "Reference" "D305"
 			(at 123.19 47.625 0)
 			(effects
@@
 			)
 		)
-		(property "Footprint" "can:DFN1006_TVS"
+		(property "Footprint" "led-matrix:DFN1006_TVS"
 			(at 123.19 50.8 0)
 			(effects
@@
 			(project "MainBoard"
 				(path "/ac576ee3-ac6f-4244-babf-9af36c7a7db3/5232c3be-bd03-4015-929e-0effd1f09850"
-					(reference "D?")
+					(reference "D305")
 					(unit 1)
 				)
@@
 		(dnp no)
 		(fields_autoplaced yes)
-		(property "Reference" "#PWR011"
+		(property "Reference" "#PWR0303"
 			(at 27.94 78.74 0)
 			(effects
@@
 			(project "MainBoard"
 				(path "/ac576ee3-ac6f-4244-babf-9af36c7a7db3/5232c3be-bd03-4015-929e-0effd1f09850"
-					(reference "#PWR011")
-					(unit 1)
-				)
+					(reference "#PWR0303")
+					(unit 1)
+				)

Commit message: dump pcb
Connections:
- net USB_SHIELD: now reaches J301.S1 (SHIELD), R303.1
Other:
- moved on the sheet: R303
Changed lines of the file:
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@@
 	(wire
 		(pts
-			(xy 20.32 68.58) (xy 20.32 72.39)
+			(xy 20.32 68.58) (xy 20.32 76.2)
 		)
 		(stroke
@@
 	(wire
 		(pts
-			(xy 20.32 80.01) (xy 20.32 82.55)
+			(xy 20.32 83.82) (xy 20.32 86.36)
 		)
 		(stroke
@@
 		)
 	)
+	(label "USB_SHIELD"
+		(at 20.32 74.93 90)
+		(fields_autoplaced yes)
+		(effects
+			(font
+				(size 0.65 0.65)
+			)
+			(justify left bottom)
+		)
+	)
 	(hierarchical_label "USB_D-"
 		(shape bidirectional)
@@
 	(symbol
 		(lib_id "Device:R")
-		(at 20.32 76.2 0)
+		(at 20.32 80.01 0)
 		(unit 1)
 		(exclude_from_sim no)
@@
 		(fields_autoplaced yes)
 		(property "Reference" "R303"
-			(at 22.86 74.9299 0)
+			(at 22.86 78.7399 0)
 			(effects
 				(font
@@
 		)
 		(property "Value" "0R"
-			(at 22.86 77.4699 0)
+			(at 22.86 81.2799 0)
 			(effects
 				(font
@@
 		)
 		(property "Footprint" "Resistor_SMD:R_0603_1608Metric"
-			(at 18.542 76.2 90)
+			(at 18.542 80.01 90)
 			(effects
 				(font
@@
 		)
 		(property "Datasheet" "~"
-			(at 20.32 76.2 0)
+			(at 20.32 80.01 0)
 			(effects
 				(font
@@
 		)
 		(property "Description" "Resistor"
-			(at 20.32 76.2 0)
+			(at 20.32 80.01 0)
 			(effects
 				(font
@@
 		)
 		(property "LCSC" "C21189"
-			(at 20.32 76.2 0)
+			(at 20.32 80.01 0)
 			(effects
 				(font
@@
 	(symbol
 		(lib_id "power:GND")
-		(at 20.32 82.55 0)
+		(at 20.32 86.36 0)
 		(unit 1)
 		(exclude_from_sim no)
@@
 		(fields_autoplaced yes)
 		(property "Reference" "#PWR0304"
-			(at 20.32 88.9 0)
+			(at 20.32 92.71 0)
 			(effects
 				(font
@@
 		)
 		(property "Value" "GND"
-			(at 20.32 87.63 0)
+			(at 20.32 91.44 0)
 			(effects
 				(font
@@
 		)
 		(property "Footprint" ""
-			(at 20.32 82.55 0)
+			(at 20.32 86.36 0)
 			(effects
 				(font
@@
 		)
 		(property "Datasheet" ""
-			(at 20.32 82.55 0)
+			(at 20.32 86.36 0)
 			(effects
 				(font
@@
 		)
 		(property "Description" "Power symbol creates a global label with name \"GND\" , ground"
-			(at 20.32 82.55 0)
-			(effects
-				(font
+			(at 20.32 86.36 0)
+			(effects
+				(font

Commit message: MainBoard: fixes, simplify, BOM optimize, DRC fixes, ERC fixes
Parts:
- J301: now left out of the parts list
Changed lines of the file:
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@@
 		(unit 1)
 		(exclude_from_sim no)
-		(in_bom yes)
+		(in_bom no)
 		(on_board yes)
 		(dnp no)
