File: pcb/MainBoard/audio.kicad_sch (KiCad schematic)
At the start: 6 parts

Commit message: pcb: main board - contd
Parts:
- J?: footprint (none) -> led-matrix:3.5mm-audio-jack; symbol Connector_Audio:AudioJack3_Ground -> Connector_Audio:AudioJack3
Connections:
- net GND: no longer J?.G
Changed lines of the file:
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@@
-	)
-	(junction
-		(at 130.81 52.07)
-		(diameter 0)
-		(color 0 0 0 0)
 	)
 	(junction
@@
 	(wire
 		(pts
-			(xy 130.81 41.91) (xy 130.81 52.07)
-		)
-		(stroke
-			(width 0)
-			(type default)
-		)
-	)
-	(wire
-		(pts
 			(xy 83.82 60.96) (xy 104.14 60.96)
 		)
@@
 	(wire
 		(pts
-			(xy 140.97 41.91) (xy 130.81 41.91)
-		)
-		(stroke
-			(width 0)
-			(type default)
-		)
-	)
-	(wire
-		(pts
 			(xy 133.35 46.99) (xy 135.89 46.99)
 		)
@@
 			(width 0)
 			(type default)
-		)
-	)
-	(text_box "TODO: select footprint"
-		(exclude_from_sim no)
-		(at 134.62 34.29 0)
-		(size 30.48 3.81)
-		(stroke
-			(width -0.0001)
-			(type default)
-		)
-		(fill
-			(type none)
-		)
-		(effects
-			(font
-				(size 1.27 1.27)
-			)
-			(justify left top)
 		)
 	)
@@
 	)
 	(symbol
-		(lib_id "Connector_Audio:AudioJack3_Ground")
+		(lib_id "Connector_Audio:AudioJack3")
 		(at 140.97 49.53 180)
 		(unit 1)
@@
 			)
 		)
-		(property "Footprint" ""
+		(property "Footprint" "led-matrix:3.5mm-audio-jack"
 			(at 140.97 49.53 0)
 			(effects
@@
 			)
 		)
-		(property "Description" "Audio Jack, 3 Poles (Stereo / TRS), Grounded Sleeve"
+		(property "Description" "Audio Jack, 3 Poles (Stereo / TRS)"
 			(at 140.97 49.53 0)
 			(effects
@@
 		(pin "R"
 		)
-		(pin "G"
-		)
 		(pin "S"

Commit message: sd card bullshit
Other:
- note added: "220R is VERY loud"
Changed lines of the file:
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@@
+		)
+	)
+	(text "220R is VERY loud"
+		(exclude_from_sim no)
+		(at 60.96 35.814 0)
+		(effects
+			(font
+				(size 1.27 1.27)
+			)
 		)
 	)

Commit message: pcb progress
Parts:
- R801: renamed from R?; value 220R -> 470R; footprint Resistor_SMD:R_0402_1005Metric -> Resistor_SMD:R_0603_1608Metric; LCSC C25091 -> C23179
- gave numbers to parts that had none: 5
Changed lines of the file:
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@@
 		(dnp no)
 		(fields_autoplaced yes)
-		(property "Reference" "C?"
+		(property "Reference" "C801"
 			(at 93.98 39.37 90)
 			(effects
@@
 			(project "MainBoard"
 				(path "/ac576ee3-ac6f-4244-babf-9af36c7a7db3/904908f8-cc64-4489-8602-62e4a247065b"
-					(reference "C?")
+					(reference "C801")
 					(unit 1)
 				)
@@
 		(on_board yes)
 		(dnp no)
-		(property "Reference" "J?"
+		(property "Reference" "J801"
 			(at 148.59 47.6249 0)
 			(effects
@@
 			(project "MainBoard"
 				(path "/ac576ee3-ac6f-4244-babf-9af36c7a7db3/904908f8-cc64-4489-8602-62e4a247065b"
-					(reference "J?")
+					(reference "J801")
 					(unit 1)
 				)
@@
 		(dnp no)
 		(fields_autoplaced yes)
-		(property "Reference" "#PWR057"
+		(property "Reference" "#PWR0802"
 			(at 77.47 72.39 0)
 			(effects
@@
 			(project "MainBoard"
 				(path "/ac576ee3-ac6f-4244-babf-9af36c7a7db3/904908f8-cc64-4489-8602-62e4a247065b"
-					(reference "#PWR057")
+					(reference "#PWR0802")
 					(unit 1)
 				)
@@
 		(on_board yes)
 		(dnp no)
-		(property "Reference" "R?"
+		(property "Reference" "R802"
 			(at 86.36 53.3399 0)
 			(effects
@@
 			(project "MainBoard"
 				(path "/ac576ee3-ac6f-4244-babf-9af36c7a7db3/904908f8-cc64-4489-8602-62e4a247065b"
-					(reference "R?")
+					(reference "R802")
 					(unit 1)
 				)
@@
 		(on_board yes)
 		(dnp no)
-		(property "Reference" "R?"
+		(property "Reference" "R803"
 			(at 106.68 53.3399 0)
 			(effects
@@
 			(project "MainBoard"
 				(path "/ac576ee3-ac6f-4244-babf-9af36c7a7db3/904908f8-cc64-4489-8602-62e4a247065b"
-					(reference "R?")
+					(reference "R803")
 					(unit 1)
 				)
@@
 		(dnp no)
 		(fields_autoplaced yes)
-		(property "Reference" "C?"
+		(property "Reference" "C802"
 			(at 73.66 53.3399 0)
 			(effects
@@
 			(project "MainBoard"
 				(path "/ac576ee3-ac6f-4244-babf-9af36c7a7db3/904908f8-cc64-4489-8602-62e4a247065b"
-					(reference "C?")
+					(reference "C802")
 					(unit 1)
 				)
@@
 		(dnp no)
 		(fields_autoplaced yes)
-		(property "Reference" "R?"
+		(property "Reference" "R801"
 			(at 62.23 40.64 90)
 			(effects
@@
 			)
 		)
-		(property "Value" "220R"
+		(property "Value" "470R"
 			(at 62.23 43.18 90)
 			(effects
@@
 			)
 		)
-		(property "Footprint" "Resistor_SMD:R_0402_1005Metric"
+		(property "Footprint" "Resistor_SMD:R_0603_1608Metric"
 			(at 62.23 45.212 90)
 			(effects
@@
 			)
 		)
-		(property "LCSC" "C25091"
+		(property "LCSC" "C23179"
 			(at 62.23 46.99 0)
 			(effects
@@
 			(project "MainBoard"
 				(path "/ac576ee3-ac6f-4244-babf-9af36c7a7db3/904908f8-cc64-4489-8602-62e4a247065b"
-					(reference "R?")
+					(reference "R801")
 					(unit 1)
 				)
@@
 		(dnp no)
 		(fields_autoplaced yes)
-		(property "Reference" "#PWR058"
+		(property "Reference" "#PWR0801"
 			(at 130.81 62.23 0)
 			(effects
@@
 			(project "MainBoard"
 				(path "/ac576ee3-ac6f-4244-babf-9af36c7a7db3/904908f8-cc64-4489-8602-62e4a247065b"
-					(reference "#PWR058")
-					(unit 1)
-				)
+					(reference "#PWR0801")
+					(unit 1)
+				)

Commit message: MainBoard: fixes, simplify, BOM optimize, DRC fixes, ERC fixes
Parts:
- C802: LCSC C307331 -> C1525
- J801: now left out of the parts list
Changed lines of the file:
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@@
 		(unit 1)
 		(exclude_from_sim no)
-		(in_bom yes)
+		(in_bom no)
 		(on_board yes)
 		(dnp no)
@@
 			)
 		)
-		(property "LCSC" "C307331"
+		(property "LCSC" "C1525"
 			(at 69.85 54.61 0)
 			(effects

Commit message: pcb: fixes, improvements
Parts:
- R801: value 470R -> 220R; LCSC C23179 -> C22962
Other:
- note added: "NOTE: 220R is VERY loud"
- note removed: "220R is VERY loud"
Changed lines of the file:
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@@
 		)
 	)
-	(text "220R is VERY loud"
-		(exclude_from_sim no)
-		(at 60.96 35.814 0)
+	(text "NOTE: 220R is VERY loud"
+		(exclude_from_sim no)
+		(at 54.864 34.798 0)
 		(effects
 			(font
@@
 			)
 		)
-		(property "Value" "470R"
+		(property "Value" "220R"
 			(at 62.23 43.18 90)
 			(effects
@@
 			)
 		)
-		(property "LCSC" "C23179"
+		(property "LCSC" "C22962"
 			(at 62.23 46.99 0)
 			(effects
