File: pcb/MainBoard/can.kicad_sch (KiCad schematic)
At the start: 5 parts

Commit message: pcb progress
Parts:
- D601, D602: renamed from D?; footprint can:DFN1006_TVS -> led-matrix:DFN1006_TVS
- gave numbers to parts that had none: 3
Changed lines of the file:
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@@
 		(on_board yes)
 		(dnp no)
-		(property "Reference" "R?"
+		(property "Reference" "R601"
 			(at 110.49 62.2299 0)
 			(effects
@@
 			(project "MainBoard"
 				(path "/ac576ee3-ac6f-4244-babf-9af36c7a7db3/085d11a9-fbb6-4cf1-879a-d3aa30071fa1"
-					(reference "R?")
+					(reference "R601")
 					(unit 1)
 				)
@@
 		(dnp no)
 		(fields_autoplaced yes)
-		(property "Reference" "#PWR049"
+		(property "Reference" "#PWR0601"
 			(at 130.81 57.15 0)
 			(effects
@@
 			(project "MainBoard"
 				(path "/ac576ee3-ac6f-4244-babf-9af36c7a7db3/085d11a9-fbb6-4cf1-879a-d3aa30071fa1"
-					(reference "#PWR049")
+					(reference "#PWR0601")
 					(unit 1)
 				)
@@
 		(dnp no)
 		(fields_autoplaced yes)
-		(property "Reference" "C?"
+		(property "Reference" "C601"
 			(at 152.4 57.1499 0)
 			(effects
@@
 			(project "MainBoard"
 				(path "/ac576ee3-ac6f-4244-babf-9af36c7a7db3/085d11a9-fbb6-4cf1-879a-d3aa30071fa1"
-					(reference "C?")
+					(reference "C601")
 					(unit 1)
 				)
@@
 		(dnp no)
 		(fields_autoplaced yes)
-		(property "Reference" "#PWR053"
+		(property "Reference" "#PWR0603"
 			(at 213.36 80.01 0)
 			(effects
@@
 			(project "MainBoard"
 				(path "/ac576ee3-ac6f-4244-babf-9af36c7a7db3/085d11a9-fbb6-4cf1-879a-d3aa30071fa1"
-					(reference "#PWR053")
+					(reference "#PWR0603")
 					(unit 1)
 				)
@@
 		(dnp no)
 		(fields_autoplaced yes)
-		(property "Reference" "U?"
+		(property "Reference" "U601"
 			(at 133.0041 64.77 0)
 			(effects
@@
 			(project "MainBoard"
 				(path "/ac576ee3-ac6f-4244-babf-9af36c7a7db3/085d11a9-fbb6-4cf1-879a-d3aa30071fa1"
-					(reference "U?")
+					(reference "U601")
 					(unit 1)
 				)
@@
 		(on_board yes)
 		(dnp no)
-		(property "Reference" "D?"
+		(property "Reference" "D601"
 			(at 208.026 63.246 0)
 			(effects
@@
 			)
 		)
-		(property "Footprint" "can:DFN1006_TVS"
+		(property "Footprint" "led-matrix:DFN1006_TVS"
 			(at 203.2 64.77 0)
 			(effects
@@
 			(project "MainBoard"
 				(path "/ac576ee3-ac6f-4244-babf-9af36c7a7db3/085d11a9-fbb6-4cf1-879a-d3aa30071fa1"
-					(reference "D?")
+					(reference "D601")
 					(unit 1)
 				)
@@
 		(dnp no)
 		(fields_autoplaced yes)
-		(property "Reference" "#PWR052"
+		(property "Reference" "#PWR0604"
 			(at 130.81 97.79 0)
 			(effects
@@
 			(project "MainBoard"
 				(path "/ac576ee3-ac6f-4244-babf-9af36c7a7db3/085d11a9-fbb6-4cf1-879a-d3aa30071fa1"
-					(reference "#PWR052")
+					(reference "#PWR0604")
 					(unit 1)
 				)
@@
 		(dnp no)
 		(fields_autoplaced yes)
-		(property "Reference" "#PWR051"
+		(property "Reference" "#PWR0602"
 			(at 148.59 68.58 0)
 			(effects
@@
 			(project "MainBoard"
 				(path "/ac576ee3-ac6f-4244-babf-9af36c7a7db3/085d11a9-fbb6-4cf1-879a-d3aa30071fa1"
-					(reference "#PWR051")
+					(reference "#PWR0602")
 					(unit 1)
 				)
@@
 		(on_board yes)
 		(dnp no)
-		(property "Reference" "D?"
+		(property "Reference" "D602"
 			(at 208.026 67.056 0)
 			(effects
@@
 			)
 		)
-		(property "Footprint" "can:DFN1006_TVS"
+		(property "Footprint" "led-matrix:DFN1006_TVS"
 			(at 203.2 68.58 0)
 			(effects
@@
 			(project "MainBoard"
 				(path "/ac576ee3-ac6f-4244-babf-9af36c7a7db3/085d11a9-fbb6-4cf1-879a-d3aa30071fa1"
-					(reference "D?")
-					(unit 1)
-				)
+					(reference "D602")
+					(unit 1)
+				)

Commit message: dump pcb
Parts:
- added J601: CANConn, Connector_JST:JST_EH_S2B-EH_1x02_P2.50mm_Horizontal, symbol Connector_Generic:Conn_01x02
- added JP601: SolderJumper_2_Open, led-matrix:SolderJumper-2_Open_RoundedPad_Smol, symbol Jumper:SolderJumper_2_Open
- added R602: 120R, Resistor_SMD:R_0402_1005Metric, symbol Device:R
Connections:
- net CANH: now also J601.1 (Pin_1), R602.2
- net CANL: now also J601.2 (Pin_2), JP601.1 (A)
- new net CAN_T_R: JP601.2 (B), R602.1
Other:
- note added: "TODO: Select connector"

Commit message: MainBoard: fixes, simplify, BOM optimize, DRC fixes, ERC fixes
Parts:
- C601: LCSC C307331 -> C1525
Changed lines of the file:
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@@
 			)
 		)
-		(property "LCSC" "C307331"
+		(property "LCSC" "C1525"
 			(at 148.59 58.42 0)
 			(effects

Commit message: pcb: fixes, improvements
Parts:
- J601: footprint Connector_JST:JST_EH_S2B-EH_1x02_P2.50mm_Horizontal -> Connector_PinHeader_2.54mm:PinHeader_1x02_P2.54mm_Horizontal
Other:
- note removed: "TODO: Select connector"
Changed lines of the file:
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@@
-		)
-	)
-	(text "TODO: Select connector"
-		(exclude_from_sim no)
-		(at 176.53 112.268 0)
-		(effects
-			(font
-				(size 1.27 1.27)
-			)
 		)
 	)
@@
 			)
 		)
-		(property "Footprint" "Connector_JST:JST_EH_S2B-EH_1x02_P2.50mm_Horizontal"
+		(property "Footprint" "Connector_PinHeader_2.54mm:PinHeader_1x02_P2.54mm_Horizontal"
 			(at 173.99 104.14 0)
 			(effects
