File: pcb/MainBoard/power.kicad_sch (KiCad schematic)
At the start: 36 parts, among them U701 AMS1117-3.3, U702 INA180A1, U703 XC6206PxxxMR-Regulator_Linear, U704 CJ431

Commit message: some pcb review
Parts:
- removed C709, C710: 4u7, Capacitor_SMD:C_0805_2012Metric, symbol Device:C_Small
- removed R708: 1k8, Resistor_SMD:R_0603_1608Metric, symbol Device:R_Small
- removed R709: 120R, Resistor_SMD:R_0402_1005Metric, symbol Device:R_Small
- removed TP706: TestPoint, TestPoint:TestPoint_Pad_D1.0mm, symbol Connector:TestPoint
- removed U703: XC6206PxxxMR-Regulator_Linear, Package_TO_SOT_SMD:SOT-23, symbol kicad-keyboard-parts:XC6206PxxxMR-Regulator_Linear
- added R?: 2k, Resistor_SMD:R_0402_1005Metric, symbol Device:R_Small
- R707: value 1k -> 680R; LCSC C11702 -> C25130
Connections:
- net GND: now also R?.2
- net VREF_REF: now also R?.1
- net VREF_REG: no longer names the net of JP701.3 (B)
Other:
- note added: "TODO: add power leds"
- moved on the sheet: R706, U704

Commit message: pcb: fixes, improvements
Parts:
- added D701, D702: LED, Diode_SMD:D_0603_1608Metric, symbol PCM_SL_Devices:LED
- added R708: 680R, Resistor_SMD:R_0402_1005Metric, symbol Device:R_Small
- added R709: 2k, Resistor_SMD:R_0402_1005Metric, symbol Device:R_Small
- added R710: 470R, Resistor_SMD:R_0603_1608Metric, symbol Device:R
- added R711: 5k1, Resistor_SMD:R_0402_1005Metric, symbol Device:R_Small
- gave numbers to parts that had none: 1
Connections:
- net 3V3: now also JP701.3 (B), D701.2
- net 5V: now also D702.2
- net GND: now also R708.1, R710.1, R711.2
- net VREF_SHUNT: now also R711.1
- new net: D701.1, R708.2
- new net: D702.1, R709.1
- new net: R709.2, R710.2
Other:
- note added: "Vref should ideally be 3v3, 431's reference is 2.5V 3,3*2/2,68=2.46 1,34mA min load: 3,3/5,1=0.6mA (5-3.3)/470=3.6mA"
- note added: "~1mA"
- note removed: "TODO: add power leds"
- note removed: "how to do this? I don't know! let's try a few ways lol"
