File: pcb/LedArrayMux/LedArrayMux.kicad_pcb (KiCad board)
At the start: 2 copper layers, 50 x 50 mm, 127 parts, among them Q1 HL2304, Q10 HL2301A, Q11 HL2301A, Q12 HL2301A, Q13 HL2301A, Q14 HL2301A, Q15 HL2301A, Q16 HL2301A, Q17 HL2301A, Q18 HL2301A, Q19 HL2301A, Q2 HL2301A, Q20 HL2301A, Q21 HL2301A, Q22 HL2304, Q23 HL2304, Q24 HL2304, Q25 HL2304, Q26 HL2304, Q27 HL2304, Q28 HL2304, Q29 HL2304, Q3 HL2301A, Q30 HL2304, Q31 HL2304, Q32 HL2304, Q33 HL2304, Q34 HL2304, Q35 HL2304, Q36 HL2304, Q37 HL2304, Q38 HL2304, Q39 HL2304, Q4 HL2301A, Q40 HL2304, Q5 HL2301A, Q6 HL2301A, Q7 HL2301A, Q8 HL2301A, Q9 HL2301A, U1 74HC595D,118, U2 74HC595D,118, U7 74HC595D,118

Commit message: pcb: mux design
Parts:
- removed D1, D2, D3: KT-0805G, LED_SMD:LED_0805_2012Metric
- removed D4: KT-0805Y, LED_SMD:LED_0805_2012Metric
- removed R1, R6: 10k, PCM_Resistor_SMD_AKL:R_0603_1608Metric_Pad0.98x0.95mm
- removed R2, R5: DNP, PCM_Resistor_SMD_AKL:R_0603_1608Metric_Pad0.98x0.95mm
- removed R85, R87, R88: 220R, PCM_Resistor_SMD_AKL:R_0603_1608Metric_Pad0.98x0.95mm
- removed R86: 440R, PCM_Resistor_SMD_AKL:R_0603_1608Metric_Pad0.98x0.95mm
- removed RN1, RN2, RN3, RN4, RN5: 100R, PCM_Resistor_SMD_AKL:R_Array_Convex_4x0603
- added ?: , , F.Cu at (195.8, 46.2)
- added ?: , , F.Cu at (195.8, 93.8)
- added ?: , , F.Cu at (148.2, 46.2)
- added ?: , , F.Cu at (148.2, 93.8)
- added C4: 22uF, Capacitor_SMD:C_1206_3216Metric, F.Cu at (149.2, 56.7)
- added C6: 10u, Capacitor_SMD:C_0603_1608Metric, F.Cu at (149.0, 64.3)
- added R10: 100R, Resistor_SMD:R_0402_1005Metric, F.Cu at (176.8, 59.6)
- added R100: 150R, Resistor_SMD:R_0805_2012Metric, F.Cu at (179.2, 49.0)
- added R101: 150R, Resistor_SMD:R_0805_2012Metric, F.Cu at (170.2, 49.0)
- added R102: 150R, Resistor_SMD:R_0805_2012Metric, F.Cu at (161.2, 49.0)
- added R103: 150R, Resistor_SMD:R_0805_2012Metric, F.Cu at (152.2, 49.0)
- added R104: 150R, Resistor_SMD:R_0805_2012Metric, F.Cu at (186.1, 49.0)
- added R105: 150R, Resistor_SMD:R_0805_2012Metric, F.Cu at (177.0, 49.0)
- added R106: 150R, Resistor_SMD:R_0805_2012Metric, F.Cu at (168.0, 49.0)
- added R107: 150R, Resistor_SMD:R_0805_2012Metric, F.Cu at (159.0, 49.0)
- added R108: 150R, Resistor_SMD:R_0805_2012Metric, F.Cu at (150.0, 49.0)
- added R12: 100R, Resistor_SMD:R_0402_1005Metric, F.Cu at (167.8, 59.6)
- added R14: 100R, Resistor_SMD:R_0402_1005Metric, F.Cu at (158.8, 59.6)
- added R16: 100R, Resistor_SMD:R_0402_1005Metric, F.Cu at (192.5, 59.6)
- added R18: 100R, Resistor_SMD:R_0402_1005Metric, F.Cu at (183.5, 59.6)
- added R20: 100R, Resistor_SMD:R_0402_1005Metric, F.Cu at (174.5, 59.6)
- added R22: 100R, Resistor_SMD:R_0402_1005Metric, F.Cu at (165.5, 59.6)
- added R24: 100R, Resistor_SMD:R_0402_1005Metric, F.Cu at (156.5, 59.6)
- added R26: 100R, Resistor_SMD:R_0402_1005Metric, F.Cu at (190.2, 59.6)
- added R28: 100R, Resistor_SMD:R_0402_1005Metric, F.Cu at (181.2, 59.6)
- added R3: 100R, Resistor_SMD:R_0402_1005Metric, F.Cu at (194.8, 59.6)
- added R30: 100R, Resistor_SMD:R_0402_1005Metric, F.Cu at (172.2, 59.6)
- added R32: 100R, Resistor_SMD:R_0402_1005Metric, F.Cu at (163.2, 59.6)
- added R34: 100R, Resistor_SMD:R_0402_1005Metric, F.Cu at (154.2, 59.6)
- added R36: 100R, Resistor_SMD:R_0402_1005Metric, F.Cu at (188.0, 59.6)
- added R38: 100R, Resistor_SMD:R_0402_1005Metric, F.Cu at (179.0, 59.6)
- added R40: 100R, Resistor_SMD:R_0402_1005Metric, F.Cu at (170.0, 59.6)
- added R42: 100R, Resistor_SMD:R_0402_1005Metric, F.Cu at (161.0, 59.6)
- added R44: 100R, Resistor_SMD:R_0402_1005Metric, F.Cu at (152.0, 59.6)
- added R46: 100R, Resistor_SMD:R_0402_1005Metric, F.Cu at (192.1, 83.1)
- added R47: 100R, Resistor_SMD:R_0402_1005Metric, F.Cu at (183.1, 83.1)
- added R49: 100R, Resistor_SMD:R_0402_1005Metric, F.Cu at (174.1, 83.1)
- added R51: 100R, Resistor_SMD:R_0402_1005Metric, F.Cu at (165.1, 83.1)
- added R53: 100R, Resistor_SMD:R_0402_1005Metric, F.Cu at (156.1, 83.1)
- added R55: 100R, Resistor_SMD:R_0402_1005Metric, F.Cu at (189.8, 83.1)
- added R57: 100R, Resistor_SMD:R_0402_1005Metric, F.Cu at (180.8, 83.1)
- added R59: 100R, Resistor_SMD:R_0402_1005Metric, F.Cu at (171.8, 83.1)
- added R61: 100R, Resistor_SMD:R_0402_1005Metric, F.Cu at (162.8, 83.1)
- added R63: 100R, Resistor_SMD:R_0402_1005Metric, F.Cu at (153.8, 83.1)
- added R65: 100R, Resistor_SMD:R_0402_1005Metric, F.Cu at (187.6, 83.1)
- added R67: 100R, Resistor_SMD:R_0402_1005Metric, F.Cu at (178.6, 83.1)
- added R69: 100R, Resistor_SMD:R_0402_1005Metric, F.Cu at (169.6, 83.1)
- added R71: 100R, Resistor_SMD:R_0402_1005Metric, F.Cu at (160.6, 83.1)
- added R73: 100R, Resistor_SMD:R_0402_1005Metric, F.Cu at (151.6, 83.1)
- added R75: 100R, Resistor_SMD:R_0402_1005Metric, F.Cu at (185.3, 83.1)
- added R77: 100R, Resistor_SMD:R_0402_1005Metric, F.Cu at (176.3, 83.1)
- added R79: 100R, Resistor_SMD:R_0402_1005Metric, F.Cu at (167.3, 83.1)
- added R8: 100R, Resistor_SMD:R_0402_1005Metric, F.Cu at (185.8, 59.6)
- added R81: 100R, Resistor_SMD:R_0402_1005Metric, F.Cu at (158.3, 83.1)
- added R83: 100R, Resistor_SMD:R_0402_1005Metric, F.Cu at (149.3, 83.1)
- added R89: 150R, Resistor_SMD:R_0805_2012Metric, F.Cu at (192.8, 49.0)
- added R90: 150R, Resistor_SMD:R_0805_2012Metric, F.Cu at (183.8, 49.0)
- added R91: 150R, Resistor_SMD:R_0805_2012Metric, F.Cu at (174.8, 49.0)
- added R92: 150R, Resistor_SMD:R_0805_2012Metric, F.Cu at (165.8, 49.0)
- added R93: 150R, Resistor_SMD:R_0805_2012Metric, F.Cu at (156.8, 49.0)
- added R94: 150R, Resistor_SMD:R_0805_2012Metric, F.Cu at (190.6, 49.0)
- added R95: 150R, Resistor_SMD:R_0805_2012Metric, F.Cu at (181.5, 49.0)
- added R96: 150R, Resistor_SMD:R_0805_2012Metric, F.Cu at (172.5, 49.0)
- added R97: 150R, Resistor_SMD:R_0805_2012Metric, F.Cu at (163.5, 49.0)
- added R98: 150R, Resistor_SMD:R_0805_2012Metric, F.Cu at (154.5, 49.0)
- added R99: 150R, Resistor_SMD:R_0805_2012Metric, F.Cu at (188.3, 49.0)
- C1, C2, C7: footprint Capacitor_SMD:C_0603_1608Metric -> Resistor_SMD:R_0402_1005Metric
- moved TP2 142.0 mm to (194.2, 61.1), turned to -90 degrees
- moved TP1 141.4 mm to (195.6, 63.0), turned to -90 degrees
- moved TP3 141.1 mm to (192.0, 61.1), turned to -90 degrees
- moved TP4 140.4 mm to (189.8, 61.1), turned to -90 degrees
- moved TP5 131.8 mm to (187.5, 61.1), turned to -90 degrees
- moved TP6 131.0 mm to (185.2, 61.1), turned to -90 degrees
- moved TP7 130.3 mm to (183.0, 61.1), turned to -90 degrees
- moved TP8 129.6 mm to (180.8, 61.1), turned to -90 degrees
- moved TP10 122.1 mm to (178.5, 61.1), turned to -90 degrees
- moved TP11 121.5 mm to (176.2, 61.1), turned to -90 degrees
- moved TP9 121.3 mm to (179.9, 63.0), turned to -90 degrees
- moved TP12 121.1 mm to (174.0, 61.1), turned to -90 degrees
- moved TP13 112.0 mm to (171.8, 61.1), turned to -90 degrees
- moved TP14 111.5 mm to (169.5, 61.1), turned to -90 degrees
- moved TP18 103.1 mm to (162.8, 61.1), turned to -90 degrees
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Connections:
- Q1 pad 1: /P0 -> Net-(Q1-G)
- Q10 pad 1: /P8 -> Net-(Q10-G)
- Q11 pad 1: /P9 -> Net-(Q11-G)
- Q12 pad 1: /P10 -> Net-(Q12-G)
- Q13 pad 1: /P11 -> Net-(Q13-G)
- Q14 pad 1: /P12 -> Net-(Q14-G)
- Q15 pad 1: /P13 -> Net-(Q15-G)
- Q16 pad 1: /P14 -> Net-(Q16-G)
- Q17 pad 1: /P15 -> Net-(Q17-G)
- Q18 pad 1: /P16 -> Net-(Q18-G)
- Q19 pad 1: /P17 -> Net-(Q19-G)
- Q2 pad 1: /P0 -> Net-(Q2-G)
- Q20 pad 1: /P18 -> Net-(Q20-G)
- Q21 pad 1: /P19 -> Net-(Q21-G)
- Q22 pad 1: /P1 -> Net-(Q22-G)
- Q23 pad 1: /P2 -> Net-(Q23-G)
- Q24 pad 1: /P3 -> Net-(Q24-G)
- Q25 pad 1: /P4 -> Net-(Q25-G)
- Q26 pad 1: /P5 -> Net-(Q26-G)
- Q27 pad 1: /P6 -> Net-(Q27-G)
- Q28 pad 1: /P7 -> Net-(Q28-G)
- Q29 pad 1: /P8 -> Net-(Q29-G)
- Q3 pad 1: /P1 -> Net-(Q3-G)
- Q30 pad 1: /P9 -> Net-(Q30-G)
- Q31 pad 1: /P10 -> Net-(Q31-G)
- Q32 pad 1: /P11 -> Net-(Q32-G)
- Q33 pad 1: /P12 -> Net-(Q33-G)
- Q34 pad 1: /P13 -> Net-(Q34-G)
- Q35 pad 1: /P14 -> Net-(Q35-G)
- Q36 pad 1: /P15 -> Net-(Q36-G)
- Q37 pad 1: /P16 -> Net-(Q37-G)
- Q38 pad 1: /P17 -> Net-(Q38-G)
- Q39 pad 1: /P18 -> Net-(Q39-G)
- Q4 pad 1: /P2 -> Net-(Q4-G)
- Q40 pad 1: /P19 -> Net-(Q40-G)
- Q5 pad 1: /P3 -> Net-(Q5-G)
- Q6 pad 1: /P4 -> Net-(Q6-G)
- Q7 pad 1: /P5 -> Net-(Q7-G)
- Q8 pad 1: /P6 -> Net-(Q8-G)
- Q9 pad 1: /P7 -> Net-(Q9-G)
- R11 pad 2: /P2 -> Net-(Q4-G)
- R13 pad 2: /P3 -> Net-(Q5-G)
- R15 pad 2: /P4 -> Net-(Q6-G)
- R17 pad 2: /P5 -> Net-(Q7-G)
- R19 pad 2: /P6 -> Net-(Q8-G)
- R21 pad 2: /P7 -> Net-(Q9-G)
- R23 pad 2: /P8 -> Net-(Q10-G)
- R25 pad 2: /P9 -> Net-(Q11-G)
- R27 pad 2: /P10 -> Net-(Q12-G)
- R29 pad 2: /P11 -> Net-(Q13-G)
- R31 pad 2: /P12 -> Net-(Q14-G)
- R33 pad 2: /P13 -> Net-(Q15-G)
- R35 pad 2: /P14 -> Net-(Q16-G)
- R37 pad 2: /P15 -> Net-(Q17-G)
- R39 pad 2: /P16 -> Net-(Q18-G)
- R4 pad 2: /P0 -> Net-(Q2-G)
- R41 pad 2: /P17 -> Net-(Q19-G)
- R43 pad 2: /P18 -> Net-(Q20-G)
- R45 pad 2: /P19 -> Net-(Q21-G)
- R48 pad 1: /P1 -> Net-(Q22-G)
- R50 pad 1: /P2 -> Net-(Q23-G)
- R52 pad 1: /P3 -> Net-(Q24-G)
- R54 pad 1: /P4 -> Net-(Q25-G)
- R56 pad 1: /P5 -> Net-(Q26-G)
- R58 pad 1: /P6 -> Net-(Q27-G)
- R60 pad 1: /P7 -> Net-(Q28-G)
- R62 pad 1: /P8 -> Net-(Q29-G)
- R64 pad 1: /P9 -> Net-(Q30-G)
- R66 pad 1: /P10 -> Net-(Q31-G)
- R68 pad 1: /P11 -> Net-(Q32-G)
- R7 pad 1: /P0 -> Net-(Q1-G)
- R70 pad 1: /P12 -> Net-(Q33-G)
- R72 pad 1: /P13 -> Net-(Q34-G)
- R74 pad 1: /P14 -> Net-(Q35-G)
- R76 pad 1: /P15 -> Net-(Q36-G)
- R78 pad 1: /P16 -> Net-(Q37-G)
- R80 pad 1: /P17 -> Net-(Q38-G)
- R82 pad 1: /P18 -> Net-(Q39-G)
- R84 pad 1: /P19 -> Net-(Q40-G)
- R9 pad 2: /P1 -> Net-(Q3-G)
- U1 pad 1: Net-(RN3-R3.1) -> /P9
- U1 pad 15: Net-(RN3-R4.1) -> /P8
- U1 pad 2: Net-(RN3-R2.1) -> /P10
- U1 pad 3: Net-(RN3-R1.1) -> /P11
- U1 pad 4: Net-(RN4-R4.1) -> /P12
- U1 pad 5: Net-(RN4-R3.1) -> /P13
- U1 pad 6: Net-(RN4-R2.1) -> /P14
- U1 pad 7: Net-(RN4-R1.1) -> /P15
- U2 pad 1: Net-(RN5-R3.1) -> /P17
- U2 pad 15: Net-(RN5-R4.1) -> /P16
- U2 pad 2: Net-(RN5-R2.1) -> /P18
- U2 pad 3: Net-(RN5-R1.1) -> /P19
- U7 pad 1: Net-(RN1-R3.1) -> /P1
- U7 pad 15: Net-(RN1-R4.1) -> /P0
- U7 pad 2: Net-(RN1-R2.1) -> /P2
- U7 pad 3: Net-(RN1-R1.1) -> /P3
- U7 pad 4: Net-(RN2-R4.1) -> /P4
- U7 pad 5: Net-(RN2-R3.1) -> /P5
- U7 pad 6: Net-(RN2-R2.1) -> /P6
- U7 pad 7: Net-(RN2-R1.1) -> /P7
Routing:
- net (no net): track 97.9 -> 0.00 mm, vias 13 -> 0
- net VLED: track 8.64 -> 81.1 mm, vias 3 -> 32
- net GND: track 18.5 -> 72.2 mm, vias 13 -> 136
- net /~{OE}: track 18.7 -> 63.6 mm, vias 0 -> 3
- net /SRCLK: track 41.8 -> 75.3 mm, vias 2 -> 3
- net /P2: track 3.81 -> 37.0 mm
- net /P18: track 3.81 -> 37.0 mm
- net /P10: track 3.81 -> 35.1 mm
- net /P9: track 7.74 -> 39.0 mm
- net /~{SRCLR}: track 49.8 -> 81.0 mm, vias 5 -> 3
- net /P20: track 3.38 -> 34.2 mm
- net /P4: track 3.81 -> 34.2 mm
- net /P22: track 2.99 -> 32.6 mm
- net /P17: track 7.74 -> 37.2 mm
- net /P1: track 7.74 -> 37.2 mm
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Other:
- board text added: "+3V3"
- board text added: "+5V"
- board text added: "0"
- board text added: "1"
- board text added: "10"
- board text added: "11"
- board text added: "12"
- board text added: "13"
- board text added: "14"
- board text added: "15"
- board text added: "16"
- board text added: "17"
- board text added: "18"
- board text added: "19"
- board text added: "2"
- board text added: "3"
- board text added: "4"
- board text added: "5"
- board text added: "6"
- board text added: "7"
- board text added: "8"
- board text added: "9"
- board text added: "GND"
- board text added: "LED Matrix Driver Module"
- board text added: "RCLK"
- board text added: "Rev A, by radex, 2024"
- board text added: "SER"
- board text added: "SRCLK"
- board text added: "~{OE}"
- board text added: "~{SRCLR}"

Commit message: LedArrayMux Rev B
Parts:
- added C101: 22uF, Capacitor_SMD:C_1206_3216Metric, F.Cu at (149.1, 61.4)
- added C102: 22uF, Capacitor_SMD:C_1206_3216Metric, F.Cu at (195.2, 52.0)
- moved C6 1.85 mm to (150.6, 65.2), turned to 0 degrees
- moved TP24 0.32 mm to (151.3, 63.4)
- moved C4 0.15 mm to (149.1, 56.7)
Routing:
- net VLED: track 81.1 -> 91.9 mm, vias 32 -> 39
- net GND: track 72.2 -> 77.7 mm, vias 136 -> 140
Other:
- board text added: "JLCJLCJLCJLC"
- board text added: "Rev B, by radex, 2024"
- board text removed: "Rev A, by radex, 2024"
