File: pcb/LedArrayMux/LedArrayMux.kicad_sch (KiCad schematic)
At the start: 127 parts, among them Q1 HL2304, Q10 HL2301A, Q11 HL2301A, Q12 HL2301A, Q13 HL2301A, Q14 HL2301A, Q15 HL2301A, Q16 HL2301A, Q17 HL2301A, Q18 HL2301A, Q19 HL2301A, Q2 HL2301A, Q20 HL2301A, Q21 HL2301A, Q22 HL2304, Q23 HL2304, Q24 HL2304, Q25 HL2304, Q26 HL2304, Q27 HL2304, Q28 HL2304, Q29 HL2304, Q3 HL2301A, Q30 HL2304, Q31 HL2304, Q32 HL2304, Q33 HL2304, Q34 HL2304, Q35 HL2304, Q36 HL2304, Q37 HL2304, Q38 HL2304, Q39 HL2304, Q4 HL2301A, Q40 HL2304, Q5 HL2301A, Q6 HL2301A, Q7 HL2301A, Q8 HL2301A, Q9 HL2301A, U1 74HC595D,118, U2 74HC595D,118, U7 74HC595D,118

Commit message: pcb: mux design
Parts:
- removed R2, R5: DNP, PCM_Resistor_SMD_AKL:R_0603_1608Metric_Pad0.98x0.95mm, symbol Device:R
- removed RN1, RN2, RN3, RN4, RN5: 100R, PCM_Resistor_SMD_AKL:R_Array_Convex_4x0603, symbol PCM_Resistor_AKL:R_4x0603_Convex
- added C3, C4: 22uF, Capacitor_SMD:C_1206_3216Metric, symbol Device:C
- added C5: 100u, Capacitor_Tantalum_SMD:CP_EIA-3528-15_AVX-H, symbol Device:C_Polarized
- added C6: 10u, Capacitor_SMD:C_0603_1608Metric, symbol Device:C
- added R10, R12, R14, R16, R18, R20, R22, R24, R26, R28, R3, R30, R32, R34, R36, R38, R40, R42, R44, R46, R47, R49, R51, R53, R55, R57, R59, R61, R63, R65, R67, R69, R71, R73, R75, R77, R79, R8, R81, R83: 100R, Resistor_SMD:R_0402_1005Metric, symbol Device:R
- added R100, R101, R102, R103, R104, R105, R106, R107, R108, R89, R90, R91, R92, R93, R94, R95, R96, R97, R98, R99: 150R, Resistor_SMD:R_0805_2012Metric, symbol Device:R
- C1, C2, C7: footprint Capacitor_SMD:C_0603_1608Metric -> Resistor_SMD:R_0402_1005Metric; LCSC C14663 -> C307331
- D1, D2, D3, D4: now not fitted
- R1, R6: footprint PCM_Resistor_SMD_AKL:R_0603_1608Metric_Pad0.98x0.95mm -> Resistor_SMD:R_0402_1005Metric; LCSC C25804 -> C25744; now not fitted
- R11, R13, R15, R17, R19, R21, R23, R25, R27, R29, R31, R33, R35, R37, R39, R4, R41, R43, R45, R48, R50, R52, R54, R56, R58, R60, R62, R64, R66, R68, R7, R70, R72, R74, R76, R78, R80, R82, R84, R9: LCSC C25804 -> C25744
- R85, R87: value 220R -> 390R; footprint PCM_Resistor_SMD_AKL:R_0603_1608Metric_Pad0.98x0.95mm -> Resistor_SMD:R_0603_1608Metric; now not fitted
- R86: value 440R -> 2k2; footprint PCM_Resistor_SMD_AKL:R_0603_1608Metric_Pad0.98x0.95mm -> Resistor_SMD:R_0603_1608Metric; now not fitted
- R88: value 220R -> 1k2; footprint PCM_Resistor_SMD_AKL:R_0603_1608Metric_Pad0.98x0.95mm -> Resistor_SMD:R_0603_1608Metric; now not fitted
Connections:
- net COL_MOS_0: now also R89.1
- net COL_MOS_1: now also R94.1
- net COL_MOS_10: now also R101.1
- net COL_MOS_11: now also R106.1
- net COL_MOS_12: now also R92.1
- net COL_MOS_13: now also R97.1
- net COL_MOS_14: now also R102.1
- net COL_MOS_15: now also R107.1
- net COL_MOS_16: now also R93.1
- net COL_MOS_17: now also R98.1
- net COL_MOS_18: now also R103.1
- net COL_MOS_19: now also R108.1
- net COL_MOS_2: now also R99.1
- net COL_MOS_3: now also R104.1
- net COL_MOS_4: now also R90.1
- net COL_MOS_5: now also R95.1
- net COL_MOS_6: now also R100.1
- net COL_MOS_7: now also R105.1
- net COL_MOS_8: now also R91.1
- net COL_MOS_9: now also R96.1
- net GND: now also C3.2, C4.2, C5.2, C6.2
- net P0: now also U7.15 (QA); no longer Q1.1 (G), Q2.1 (G), R4.2, R7.1
- net P1: now also U7.1 (QB), R3.1, R46.1; no longer Q22.1 (G), Q3.1 (G), R48.1, R9.2
- net P10: now also U1.2 (QC), R10.1, R49.2; no longer Q12.1 (G), Q31.1 (G), R27.2, R66.1
- net P11: now also U1.3 (QD), R20.1, R59.2; no longer Q13.1 (G), Q32.1 (G), R29.2, R68.1
- net P12: now also U1.4 (QE), R30.1, R69.2; no longer Q14.1 (G), Q33.1 (G), R31.2, R70.1
- net P13: now also U1.5 (QF), R40.1, R79.2; no longer Q15.1 (G), Q34.1 (G), R33.2, R72.1
- net P14: now also U1.6 (QG), R12.1, R51.2; no longer Q16.1 (G), Q35.1 (G), R35.2, R74.1
- net P15: now also U1.7 (QH), R22.1, R61.2; no longer Q17.1 (G), Q36.1 (G), R37.2, R76.1
- net P16: now also U2.15 (QA); no longer Q18.1 (G), Q37.1 (G), R39.2, R78.1
- net P17: now also U2.1 (QB), R32.1, R71.2; no longer Q19.1 (G), Q38.1 (G), R41.2, R80.1
- net P18: now also U2.2 (QC), R42.1, R81.2; no longer Q20.1 (G), Q39.1 (G), R43.2, R82.1
- net P19: now also U2.3 (QD), R14.1, R53.2; no longer Q21.1 (G), Q40.1 (G), R45.2, R84.1
- net P2: now also U7.2 (QC), R16.1, R55.2; no longer Q23.1 (G), Q4.1 (G), R11.2, R50.1
- net P20: now also R24.1, R63.2
- net P21: now also R34.1, R73.2
- net P22: now also R44.1, R83.2
- net P3: now also U7.3 (QD), R26.1, R65.2; no longer Q24.1 (G), Q5.1 (G), R13.2, R52.1
- net P4: now also U7.4 (QE), R36.1, R75.2; no longer Q25.1 (G), Q6.1 (G), R15.2, R54.1
- net P5: now also U7.5 (QF), R47.2, R8.1; no longer Q26.1 (G), Q7.1 (G), R17.2, R56.1
- net P6: now also U7.6 (QG), R18.1, R57.2; no longer Q27.1 (G), Q8.1 (G), R19.2, R58.1
- net P7: now also U7.7 (QH), R28.1, R67.2; no longer Q28.1 (G), Q9.1 (G), R21.2, R60.1
- net P8: now also U1.15 (QA); no longer Q10.1 (G), Q29.1 (G), R23.2, R62.1
- net P9: now also U1.1 (QB), R38.1, R77.2; no longer Q11.1 (G), Q30.1 (G), R25.2, R64.1
- net VCC: now also C3.1, C6.1
- net VLED: now also C4.1, C5.1
- new net: Q37.1 (G), R53.1, R78.1
- new net: Q15.1 (G), R22.2, R33.2
- new net: Q11.1 (G), R20.2, R25.2
- new net: Q23.1 (G), R50.1, R65.1
- new net: Q9.1 (G), R21.2, R38.2
- new net: Q27.1 (G), R58.1, R67.1
- new net: Q30.1 (G), R59.1, R64.1
- new net: Q38.1 (G), R63.1, R80.1
- new net: Q24.1 (G), R52.1, R75.1
- new net: Q28.1 (G), R60.1, R77.1
- new net: Q14.1 (G), R12.2, R31.2
- new net: Q5.1 (G), R13.2, R36.2
- new net: Q17.1 (G), R37.2, R42.2
- new net: Q34.1 (G), R61.1, R72.1
- new net: Q12.1 (G), R27.2, R30.2
- new net: Q29.1 (G), R49.1, R62.1
- new net: Q3.1 (G), R16.2, R9.2
- new net: Q1.1 (G), R46.2, R7.1
- new net: Q22.1 (G), R48.1, R55.1
- new net: Q13.1 (G), R29.2, R40.2
- new net: Q32.1 (G), R68.1, R79.1
- new net: Q36.1 (G), R76.1, R81.1
- new net: Q21.1 (G), R44.2, R45.2
- new net: Q39.1 (G), R73.1, R82.1
- new net: Q18.1 (G), R14.2, R39.2
- new net: Q10.1 (G), R10.2, R23.2
- new net: Q4.1 (G), R11.2, R26.2
- new net: Q31.1 (G), R66.1, R69.1
- new net: Q7.1 (G), R17.2, R18.2
- new net: Q33.1 (G), R51.1, R70.1
- new net: Q35.1 (G), R71.1, R74.1
- new net: Q2.1 (G), R3.2, R4.2
- new net: Q8.1 (G), R19.2, R28.2
- new net: Q19.1 (G), R24.2, R41.2
- new net: Q40.1 (G), R83.1, R84.1
- new net: Q26.1 (G), R56.1, R57.1
- new net: Q16.1 (G), R32.2, R35.2
- new net: Q6.1 (G), R15.2, R8.2
- new net: Q20.1 (G), R34.2, R43.2
- new net: Q25.1 (G), R47.1, R54.1
- new net COL_0: R89.2
- new net COL_1: R94.2
- new net COL_10: R101.2
- new net COL_11: R106.2
- new net COL_12: R92.2
- new net COL_13: R97.2
- new net COL_14: R102.2
- new net COL_15: R107.2
- new net COL_16: R93.2
- new net COL_17: R98.2
- new net COL_18: R103.2
- new net COL_19: R108.2
- new net COL_2: R99.2
- new net COL_3: R104.2
- new net COL_4: R90.2
- new net COL_5: R95.2
- new net COL_6: R100.2
- new net COL_7: R105.2
- new net COL_8: R91.2
- new net COL_9: R96.2
Other:
- note added: "Current limiting resistors"
- note added: "Decoupling"
- note added: "Not all parallel outputs are used!"
- note added: "VCC: 3.3V VLED: 5V Aiming for 1mA for status lights"
- note removed: "(3.3-2.1)/220 = 5.5mA"
- note removed: "(5-2.8)/220 = 10mA (3.3-2.8)/220 = 2.2mA"
- note removed: "(6-2.8)/440 = 7mA (5-2.8)/440 = 5mA (3-2.8)/220 = 0.5mA"
- note removed: "Only P0-P19 are used, P20-P23 have test points only"
- note removed: "VCC: unknown, 3.3-5V VLED: unknown, likely 3-6V Aiming for 2-5mA for status LEDs"
- moved on the sheet: TP1, TP10, TP11, TP12, TP13, TP14, TP15, TP16, TP17, TP18, TP19, TP2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

Commit message: LedArrayMux Rev B
Parts:
- added C101, C102: 22uF, Capacitor_SMD:C_1206_3216Metric, symbol Device:C
Connections:
- net GND: now also C101.2, C102.2
- net VLED: now also C101.1, C102.1
Other:
- moved on the sheet: C4, C5
